Commit message: feat(urdf): add new URDF files for Wheel_leg_V1

File: source/agent_world/agent_world/assets/usd_files/Wheel_leg_V1/urdf/urdf_V4.0_cylwheel.urdf (robot description, URDF)
Before this commit: robot Wheel_leg_V1, 7 links, 6 joints
Links:
- link L_link3: geometry collision cylinder length=0.0250000003725 radius=0.0600000032506; visual mesh filename=../meshes/L_link3.STL
- link R_link3: geometry collision cylinder length=0.0250000003725 radius=0.0600000031546; visual mesh filename=../meshes/R_link3.STL
